File: OOPS-All-Knobs/OOPS-All-Knobs.kicad_pcb (KiCad board)
At the start: 2 copper layers, 226.5 x 75 mm, 181 parts, among them J1 USB_C_Receptacle_USB2.0, J2 Conn_01x03_Female, SW1 SW_SPST, SW2 SW_SPST, U1 NCP1117-3.3_SOT223, U2 W25Q128JVS, U3 RP2040TR7, U4 SRV05-4, Y1 12MHz

Commit message: Everything but the crystal
Parts:
- U1: value NCP1117-3.3_SOT223 -> XC6206PxxxMR; footprint Package_TO_SOT_SMD:SOT-89-3 -> Package_TO_SOT_SMD:SOT-23
- moved C2 3.20 mm to (65.0, 33.0), turned to -90 degrees
- moved U1 0.62 mm to (62.5, 33.7)
Routing:
- net Net-(C1-Pad1): track 4.36 -> 9.49 mm
- net +3V3: track 138.3 -> 133.7 mm
- net GND: track 100.9 -> 103.8 mm, vias 65 -> 66
