File: OOPS-All-Knobs/OOPS-All-Knobs.kicad_sch (KiCad schematic)
At the start: 180 parts, among them J1 USB_C_Receptacle_USB2.0, J2 Conn_01x03_Female, SW1 SW_SPST, SW2 SW_SPST, U1 NCP1117-3.3_SOT223, U2 W25Q128JVS, U3 RP2040TR7, U4 SRV05-4, Y1 12MHz

Commit message: Everything but the crystal
Parts:
- U1: value NCP1117-3.3_SOT223 -> XC6206PxxxMR; footprint Package_TO_SOT_SMD:SOT-89-3 -> Package_TO_SOT_SMD:SOT-23; symbol Regulator_Linear:NCP1117-3.3_SOT223 -> Regulator_Linear:XC6206PxxxMR
Changed lines of the file:
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@@
     (pin "2")
   )
-  (symbol (lib_id "Regulator_Linear:NCP1117-3.3_SOT223") (at 90.805 26.67 0) (unit 1)
+  (symbol (lib_id "Regulator_Linear:XC6206PxxxMR") (at 90.805 26.67 0) (unit 1)
     (in_bom yes) (on_board yes)
     (property "Reference" "U1" (id 0) (at 90.805 20.7985 0))
-    (property "Value" "NCP1117-3.3_SOT223" (id 1) (at 90.805 23.5736 0))
-    (property "Footprint" "Package_TO_SOT_SMD:SOT-89-3" (id 2) (at 90.805 21.59 0)
-      (effects (font (size 1.27 1.27)) hide)
+    (property "Value" "XC6206PxxxMR" (id 1) (at 90.805 23.495 0)
+      (effects (font (size 1.27 1.27)) (justify left))
+    )
+    (property "Footprint" "Package_TO_SOT_SMD:SOT-23" (id 2) (at 90.805 20.955 0)
+      (effects (font (size 1.27 1.27) italic) hide)
     )
-    (property "Datasheet" "http://www.onsemi.com/pub_link/Collateral/NCP1117-D.PDF" (id 3) (at 93.345 33.02 0)
+    (property "Datasheet" "https://www.torexsemi.com/file/xc6206/XC6206.pdf" (id 3) (at 90.805 26.67 0)
       (effects (font (size 1.27 1.27)) hide)
     )
@@
     )
     (path "/121366cb-3a8e-45f4-98d3-8d885202a353"
-      (reference "U1") (unit 1) (value "NCP1117-3.3_SOT223") (footprint "Package_TO_SOT_SMD:SOT-89-3")
+      (reference "U1") (unit 1) (value "XC6206PxxxMR") (footprint "Package_TO_SOT_SMD:SOT-23")
     )
     (path "/f45f6b32-e1fb-4a78-96d7-bf8772a80419"

Commit message: Ready for Manu!
Parts:
- C5, C6: value 27p -> 30p
- Y1: value 12MHz -> Crystal_GND24_Small; symbol Device:Crystal -> Device:Crystal_GND24_Small
Connections:
- net GND: now also Y1.2, Y1.4
- net XIN: now also Y1.3; no longer Y1.2
Changed lines of the file:
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@@
   (junction (at 176.53 50.8) (diameter 0) (color 0 0 0 0)
   )
-  (junction (at 129.54 154.94) (diameter 0) (color 0 0 0 0)
-  )
   (junction (at 187.96 86.36) (diameter 0) (color 0 0 0 0)
   )
@@
   (junction (at 225.425 154.94) (diameter 0) (color 0 0 0 0)
   )
+  (junction (at 129.54 154.94) (diameter 0) (color 0 0 0 0)
+  )
   (junction (at 151.13 76.2) (diameter 0) (color 0 0 0 0)
   )
@@
   (junction (at 100.965 26.67) (diameter 0) (color 0 0 0 0)
   )
+  (junction (at 120.015 158.115) (diameter 0) (color 0 0 0 0)
+  )
   (junction (at 220.98 78.105) (diameter 0) (color 0 0 0 0)
   )
@@
   (junction (at 132.08 102.87) (diameter 0) (color 0 0 0 0)
   )
+  (junction (at 120.015 151.13) (diameter 0) (color 0 0 0 0)
+  )
   (junction (at 265.43 101.6) (diameter 0) (color 0 0 0 0)
   )
@@
     (stroke (width 0) (type default) (color 0 0 0 0))
   )
+  (wire (pts (xy 120.015 151.13) (xy 120.015 154.94))
+    (stroke (width 0) (type default) (color 0 0 0 0))
+  )
   (wire (pts (xy 123.825 48.26) (xy 123.19 48.26))
     (stroke (width 0) (type default) (color 0 0 0 0))
@@
     (stroke (width 0) (type default) (color 0 0 0 0))
   )
+  (wire (pts (xy 129.54 154.94) (xy 136.525 154.94))
+    (stroke (width 0) (type default) (color 0 0 0 0))
+  )
   (wire (pts (xy 149.86 28.575) (xy 175.26 28.575))
     (stroke (width 0) (type default) (color 0 0 0 0))
@@
     (stroke (width 0) (type default) (color 0 0 0 0))
   )
+  (wire (pts (xy 129.54 147.32) (xy 129.54 148.59))
+    (stroke (width 0) (type default) (color 0 0 0 0))
+  )
   (wire (pts (xy 149.86 86.36) (xy 152.4 86.36))
     (stroke (width 0) (type default) (color 0 0 0 0))
@@
     (stroke (width 0) (type default) (color 0 0 0 0))
   )
-  (wire (pts (xy 120.015 156.845) (xy 120.015 154.94))
+  (wire (pts (xy 120.015 158.115) (xy 120.015 154.94))
     (stroke (width 0) (type default) (color 0 0 0 0))
   )
@@
     (stroke (width 0) (type default) (color 0 0 0 0))
   )
-  (wire (pts (xy 129.54 154.94) (xy 136.525 154.94))
+  (wire (pts (xy 125.095 154.94) (xy 129.54 154.94))
     (stroke (width 0) (type default) (color 0 0 0 0))
   )
@@
     (stroke (width 0) (type default) (color 0 0 0 0))
   )
-  (wire (pts (xy 125.095 154.94) (xy 129.54 154.94))
-    (stroke (width 0) (type default) (color 0 0 0 0))
-  )
   (wire (pts (xy 80.645 34.29) (xy 90.805 34.29))
     (stroke (width 0) (type default) (color 0 0 0 0))
@@
     (stroke (width 0) (type default) (color 0 0 0 0))
   )
+  (wire (pts (xy 132.08 151.13) (xy 132.08 158.115))
+    (stroke (width 0) (type default) (color 0 0 0 0))
+  )
   (wire (pts (xy 259.08 52.07) (xy 259.08 50.8))
     (stroke (width 0) (type default) (color 0 0 0 0))
@@
     (stroke (width 0) (type default) (color 0 0 0 0))
   )
-  (wire (pts (xy 120.015 147.32) (xy 120.015 154.94))
+  (wire (pts (xy 120.015 147.32) (xy 120.015 151.13))
     (stroke (width 0) (type default) (color 0 0 0 0))
   )
@@
     (stroke (width 0) (type default) (color 0 0 0 0))
   )
+  (wire (pts (xy 132.08 158.115) (xy 120.015 158.115))
+    (stroke (width 0) (type default) (color 0 0 0 0))
+  )
   (wire (pts (xy 142.24 86.36) (xy 144.78 86.36))
     (stroke (width 0) (type default) (color 0 0 0 0))
@@
     (stroke (width 0) (type default) (color 0 0 0 0))
   )
+  (wire (pts (xy 129.54 153.67) (xy 129.54 154.94))
+    (stroke (width 0) (type default) (color 0 0 0 0))
+  )
   (wire (pts (xy 213.36 50.8) (xy 214.63 50.8))
     (stroke (width 0) (type default) (color 0 0 0 0))
@@
     (stroke (width 0) (type default) (color 0 0 0 0))
   )
+  (wire (pts (xy 120.015 151.13) (xy 127 151.13))
+    (stroke (width 0) (type default) (color 0 0 0 0))
+  )
   (wire (pts (xy 256.54 35.56) (xy 256.54 60.96))
     (stroke (width 0) (type default) (color 0 0 0 0))
@@
     (pin "1")
   )
-  (symbol (lib_id "power:GND") (at 120.015 156.845 0) (unit 1)
+  (symbol (lib_id "power:GND") (at 120.015 158.115 0) (unit 1)
     (in_bom yes) (on_board yes) (fields_autoplaced)
-    (property "Reference" "#PWR057" (id 0) (at 120.015 163.195 0)
+    (property "Reference" "#PWR057" (id 0) (at 120.015 164.465 0)
       (effects (font (size 1.27 1.27)) hide)
     )
-    (property "Value" "GND" (id 1) (at 120.015 161.4075 0))
-    (property "Footprint" "" (id 2) (at 120.015 156.845 0)
+    (property "Value" "GND" (id 1) (at 120.015 162.6775 0))
+    (property "Footprint" "" (id 2) (at 120.015 158.115 0)
       (effects (font (size 1.27 1.27)) hide)
     )
-    (property "Datasheet" "" (id 3) (at 120.015 156.845 0)
+    (property "Datasheet" "" (id 3) (at 120.015 158.115 0)
       (effects (font (size 1.27 1.27)) hide)
     )
@@
     (in_bom yes) (on_board yes) (fields_autoplaced)
     (property "Reference" "C6" (id 0) (at 122.5486 149.4114 90))
-    (property "Value" "27p" (id 1) (at 122.5486 152.1865 90))
+    (property "Value" "30p" (id 1) (at 122.5486 152.1865 90))
     (property "Footprint" "Capacitor_SMD:C_0402_1005Metric" (id 2) (at 122.555 154.94 0)
       (effects (font (size 1.27 1.27)) hide)
@@
     (pin "2")
   )
-  (symbol (lib_id "Device:Crystal") (at 129.54 151.13 270) (unit 1)
+  (symbol (lib_id "Device:Crystal_GND24_Small") (at 129.54 151.13 270) (unit 1)
     (in_bom yes) (on_board yes)
     (property "Reference" "Y1" (id 0) (at 132.8674 150.2215 90)
       (effects (font (size 1.27 1.27)) (justify left))
     )
-    (property "Value" "12MHz" (id 1) (at 126.365 145.415 90)
+    (property "Value" "Crystal_GND24_Small" (id 1) (at 132.08 152.4 90)
       (effects (font (size 1.27 1.27)) (justify left))
     )
@@
     (pin "1")
     (pin "2")
+    (pin "3")
+    (pin "4")
   )
   (symbol (lib_id "power:GND") (at 160.02 76.2 0) (unit 1)
@@
     (in_bom yes) (on_board yes) (fields_autoplaced)
     (property "Reference" "C5" (id 0) (at 122.5613 141.7914 90))
-    (property "Value" "27p" (id 1) (at 122.5613 144.5665 90))
+    (property "Value" "30p" (id 1) (at 122.5613 144.5665 90))
     (property "Footprint" "Capacitor_SMD:C_0402_1005Metric" (id 2) (at 122.555 147.32 0)
       (effects (font (size 1.27 1.27)) hide)
@@
     )
     (path "/eecfaddf-fe1d-4b76-bad9-b3bf6583dd17"
-      (reference "C5") (unit 1) (value "27p") (footprint "Capacitor_SMD:C_0402_1005Metric")
+      (reference "C5") (unit 1) (value "30p") (footprint "Capacitor_SMD:C_0402_1005Metric")
     )
     (path "/69133ab9-30ae-473e-99f8-2d3bda574ee2"
-      (reference "C6") (unit 1) (value "27p") (footprint "Capacitor_SMD:C_0402_1005Metric")
+      (reference "C6") (unit 1) (value "30p") (footprint "Capacitor_SMD:C_0402_1005Metric")
     )
     (path "/9a4070c7-eedc-4dec-b0b5-9804ebbb050f"
@@
     )
     (path "/ba590642-459a-4589-bf88-8193edcd8748"
-      (reference "Y1") (unit 1) (value "12MHz") (footprint "Crystal:Crystal_SMD_3225-4Pin_3.2x2.5mm")
+      (reference "Y1") (unit 1) (value "Crystal_GND24_Small") (footprint "Crystal:Crystal_SMD_3225-4Pin_3.2x2.5mm")
     )
   )
